File: minRead_pcb/minRead_pcb.kicad_pcb (KiCad board)
At the start: 2 copper layers, 64.5 x 120.5 mm, 119 parts, among them J1 USB_C_Receptacle, J2 FH34SRJ-24S-0.5SH_50_, J3 FH34SRJ-6S-0.5SH_50_, J5 Conn_01x02, J6 PPTC052LFBN-RC, J7 Micro_SD_Card, Q1 FS8205A, Q2 IRLML6402, Q3 IRLML6402, Q4 BSS138, Q5 BSS138, Q6 BSS138, Q7 IRLML6402, Q8 IRLML6402, Q9 MMBT3904, SW1 SW_Push, SW10 SW_Push, SW12 SW_Push, SW2 SW_Push, SW3 SW_Push, SW4 SW_Push, SW5 SW_Push, SW6 SW_Push, SW7 SW_Push, SW8 SW_Push, SW9 SW_Push, U1 TPD4E1U06DBVR, U2 AP3012, U3 AP2112K-3.3, U4 ESP32-S3-WROOM-1, U5 DW01A, U6 TPD4E1U06DBVR, U7 MCP73832-2-OT

Commit message: current prototype
Parts:
- removed R17: 100, Resistor_SMD:R_0805_2012Metric_Pad1.20x1.40mm_HandSolder
- added G***: LOGO, LOGO, F.Cu at (145.5, 58.5)
- added G***: LOGO, LOGO, B.Cu at (151.0, 58.5)
- C8: value 0.1u -> 1u
- C9: value 1u -> 4.7u
- J6: moved to B.Cu
- moved U3 42.6 mm to (155.6, 123.2)
- moved C4 40.6 mm to (156.6, 128.2), turned to -90 degrees
- moved C6 40.0 mm to (152.6, 122.7), turned to -90 degrees
- moved CR1 39.0 mm to (149.0, 146.0), turned to 90 degrees
- moved J1 37.2 mm to (158.5, 145.5)
- moved D1 37.2 mm to (153.2, 140.0)
- moved D2 37.0 mm to (153.5, 132.0)
- moved R38 37.0 mm to (152.5, 135.5)
- moved Q2 36.1 mm to (156.5, 135.0), turned to -90 degrees
- moved J3 33.3 mm to (119.0, 136.5)
- moved C12 33.1 mm to (118.5, 119.6)
- moved C9 33.1 mm to (118.5, 131.0)
- moved D7 33.1 mm to (119.0, 128.6)
- moved L2 33.1 mm to (120.5, 125.0)
- moved Q5 33.1 mm to (122.5, 119.5)
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Connections:
- CR1 pad 1: USB_VBUS -> /VBUS_PRE
- D1 pad 2: Net-(D1-A) -> /VBUS_PRE
- J1 pad A4: Net-(D1-A) -> /VBUS_PRE
- J1 pad A9: Net-(D1-A) -> /VBUS_PRE
- J1 pad B4: Net-(D1-A) -> /VBUS_PRE
- J1 pad B9: Net-(D1-A) -> /VBUS_PRE
- Q8 pad 2: Net-(Q8-S) -> P+
Routing:
- net C-: track 97.0 -> 155.9 mm, vias 0 -> 4
- net COOL_TOGGLE: track 106.9 -> 160.9 mm
- net 3V3: track 337.6 -> 390.7 mm
- net LED_SW: track 90.8 -> 143.1 mm
- net CC1: track 11.0 -> 54.6 mm, vias 2 -> 3
- net Net-(J1-SHIELD): track 23.3 -> 62.1 mm, vias 0 -> 1
- net CHG_STATUS: track 83.0 -> 118.0 mm
- net CC2: track 20.0 -> 51.4 mm
- net DN: track 150.5 -> 178.5 mm, vias 5 -> 4
- net WARM_TOGGLE: track 114.4 -> 142.3 mm
- net W-: track 90.2 -> 114.4 mm, vias 2 -> 5
- net LED_PWR: track 80.5 -> 103.8 mm
- net DP: track 153.3 -> 176.3 mm
- net /VBUS_PRE: track 0.00 -> 22.0 mm
- net LED_SENSE: track 84.2 -> 102.6 mm
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Other:
- outline, holes or cut-outs redrawn
- board text added: "24 1"
- board text added: "24-pin epaper slots here!"
- board text added: "3v3"
- board text added: "6-pin LED!"
- board text added: "ESP32-S3 WROOM"
- board text added: "G"
- board text added: "Thank you! - Ian C"
- board text added: "^"
- board text added: "cat by @tomisit0"
- board text added: "microSD if you please"
