File: minRead_pcb/minRead_pcb.kicad_sch (KiCad schematic)
At the start: 119 parts, among them J1 USB_C_Receptacle, J2 FH34SRJ-24S-0.5SH_50_, J3 FH34SRJ-6S-0.5SH_50_, J5 Conn_01x02, J6 PPTC052LFBN-RC, J7 Micro_SD_Card, Q1 FS8205A, Q2 IRLML6402, Q3 IRLML6402, Q4 BSS138, Q5 BSS138, Q6 BSS138, Q7 IRLML6402, Q8 IRLML6402, Q9 MMBT3904, SW1 SW_Push, SW10 SW_Push, SW12 SW_Push, SW2 SW_Push, SW3 SW_Push, SW4 SW_Push, SW5 SW_Push, SW6 SW_Push, SW7 SW_Push, SW8 SW_Push, SW9 SW_Push, U1 TPD4E1U06DBVR, U2 AP3012, U3 AP2112K-3.3, U4 ESP32-S3-WROOM-1, U5 DW01A, U6 TPD4E1U06DBVR, U7 MCP73832-2-OT

Commit message: current prototype
Parts:
- removed R17: 100, Resistor_SMD:R_0805_2012Metric_Pad1.20x1.40mm_HandSolder, symbol Device:R
- C8: value 0.1u -> 1u
- C9: value 1u -> 4.7u
Connections:
- net P+: now also Q8.2 (S)
- net USB_VBUS: no longer CR1.1 (I/O)
- net VBUS_PRE: now reaches D1.2 (A), J1.A4 (VBUS), J1.A9 (VBUS), J1.B4 (VBUS), J1.B9 (VBUS)
- net VBUS_PRE: now also CR1.1 (I/O)
Other:
- moved on the sheet: D1
Changed lines of the file:
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@@
 	)
 	(junction
+		(at 285.75 284.48)
+		(diameter 0)
+		(color 0 0 0 0)
+	)
+	(junction
 		(at 148.59 323.85)
 		(diameter 0)
@@
 	(wire
 		(pts
+			(xy 52.07 30.48) (xy 48.26 30.48)
+		)
+		(stroke
+			(width 0)
+			(type default)
+		)
+	)
+	(wire
+		(pts
 			(xy 148.59 323.85) (xy 115.57 323.85)
 		)
@@
 	(wire
 		(pts
-			(xy 73.66 156.21) (xy 76.2 156.21)
-		)
-		(stroke
-			(width 0)
-			(type default)
-		)
-	)
-	(wire
-		(pts
 			(xy 424.18 111.76) (xy 431.8 111.76)
 		)
@@
 	(wire
 		(pts
-			(xy 55.88 30.48) (xy 62.23 30.48)
+			(xy 59.69 30.48) (xy 62.23 30.48)
 		)
 		(stroke
@@
 	(wire
 		(pts
+			(xy 285.75 284.48) (xy 287.02 284.48)
+		)
+		(stroke
+			(width 0)
+			(type default)
+		)
+	)
+	(wire
+		(pts
 			(xy 292.1 173.99) (xy 292.1 182.88)
 		)
@@
 	(wire
 		(pts
-			(xy 284.48 284.48) (xy 287.02 284.48)
+			(xy 284.48 284.48) (xy 285.75 284.48)
 		)
 		(stroke
@@
 	(wire
 		(pts
-			(xy 62.23 156.21) (xy 66.04 156.21)
+			(xy 62.23 156.21) (xy 76.2 156.21)
 		)
 		(stroke
@@
 		)
 	)
+	(label "VBUS_PRE"
+		(at 49.53 30.48 90)
+		(effects
+			(font
+				(size 1.27 1.27)
+			)
+			(justify left bottom)
+		)
+	)
 	(label "PREVGL"
 		(at 49.53 313.69 0)
@@
 		)
 	)
+	(label "VBUS_PRE"
+		(at 36.83 121.92 180)
+		(effects
+			(font
+				(size 1.27 1.27)
+			)
+			(justify right bottom)
+		)
+	)
 	(label "CMD"
 		(at 439.42 83.82 180)
@@
 		)
 	)
-	(global_label "USB_VBUS"
-		(shape input)
-		(at 36.83 121.92 180)
-		(fields_autoplaced yes)
-		(effects
-			(font
-				(size 1.27 1.27)
-			)
-			(justify right)
-		)
-		(property "Intersheetrefs" "${INTERSHEET_REFS}"
-			(at 24.1686 121.92 0)
-			(effects
-				(font
-					(size 1.27 1.27)
-				)
-				(justify right)
-				(hide yes)
-			)
-		)
-	)
 	(global_label "EPD_DC"
 		(shape input)
@@
 			)
 		)
-		(property "Value" "0.1u"
+		(property "Value" "1u"
 			(at 196.85 105.4099 0)
 			(effects
@@
 	)
 	(symbol
+		(lib_id "power:PWR_FLAG")
+		(at 285.75 284.48 0)
+		(unit 1)
+		(exclude_from_sim no)
+		(in_bom yes)
+		(on_board yes)
+		(dnp no)
+		(fields_autoplaced yes)
+		(property "Reference" "#FLG05"
+			(at 285.75 282.575 0)
+			(effects
+				(font
+					(size 1.27 1.27)
+				)
+				(hide yes)
+			)
+		)
+		(property "Value" "PWR_FLAG"
+			(at 285.75 279.4 0)
+			(effects
+				(font
+					(size 1.27 1.27)
+				)
+			)
+		)
+		(property "Footprint" ""
+			(at 285.75 284.48 0)
+			(effects
+				(font
+					(size 1.27 1.27)
+				)
+				(hide yes)
+			)
+		)
+		(property "Datasheet" "~"
+			(at 285.75 284.48 0)
+			(effects
+				(font
+					(size 1.27 1.27)
+				)
+				(hide yes)
+			)
+		)
+		(property "Description" "Special symbol for telling ERC where power comes from"
+			(at 285.75 284.48 0)
+			(effects
+				(font
+					(size 1.27 1.27)
+				)
+				(hide yes)
+			)
+		)
+		(pin "1"
+		)
+		(instances
+			(project "minRead_pcb"
+				(path "/2fbd4c8f-b784-4d80-b374-4947df99a9bf"
+					(reference "#FLG05")
+					(unit 1)
+				)
+			)
+		)
+	)
+	(symbol
 		(lib_id "Mechanical:MountingHole_Pad")
 		(at 364.49 262.89 0)
@@
 			)
 		)
-		(property "Value" "1u"
+		(property "Value" "4.7u"
 			(at 340.614 270.51 90)
 			(effects
@@
 	(symbol
 		(lib_id "Diode:MBR0530")
-		(at 52.07 30.48 180)
+		(at 55.88 30.48 180)
 		(unit 1)
 		(exclude_from_sim no)
@@
 		(fields_autoplaced yes)
 		(property "Reference" "D1"
-			(at 52.3875 24.13 0)
+			(at 56.1975 24.13 0)
 			(effects
 				(font
@@
 		)
 		(property "Value" "MBR0530"
-			(at 52.3875 26.67 0)
+			(at 56.1975 26.67 0)
 			(effects
 				(font
@@
 		)
 		(property "Footprint" "Diode_SMD:D_SOD-123"
-			(at 52.07 26.035 0)
+			(at 55.88 26.035 0)
 			(effects
 				(font
@@
 		)
 		(property "Datasheet" "http://www.mccsemi.com/up_pdf/MBR0520~MBR0580(SOD123).pdf"
-			(at 52.07 30.48 0)
+			(at 55.88 30.48 0)
 			(effects
 				(font
@@
 		)
 		(property "Description" "30V 0.5A Schottky Power Rectifier Diode, SOD-123"
-			(at 52.07 30.48 0)
+			(at 55.88 30.48 0)
 			(effects
 				(font
@@
 					(unit 1)
 				)
-			)
-		)
-	)
-	(symbol
-		(lib_id "Device:R")
-		(at 69.85 156.21 90)
-		(unit 1)
-		(exclude_from_sim no)
-		(in_bom yes)
-		(on_board yes)
-		(dnp no)
-		(property "Reference" "R17"
-			(at 69.85 149.86 90)
-			(effects
-				(font
-					(size 1.27 1.27)
-				)
-			)
-		)
-		(property "Value" "100"
-			(at 69.85 152.4 90)
-			(effects
-				(font
-					(size 1.27 1.27)
-				)
-			)
-		)
-		(property "Footprint" "Resistor_SMD:R_0805_2012Metric_Pad1.20x1.40mm_HandSolder"
-			(at 69.85 157.988 90)
-			(effects
-				(font
-					(size 1.27 1.27)
-				)
-				(hide yes)
-			)
-		)
-		(property "Datasheet" "~"
-			(at 69.85 156.21 0)
-			(effects
-				(font
-					(size 1.27 1.27)
-				)
-				(hide yes)
-			)
-		)
-		(property "Description" "Resistor"
-			(at 69.85 156.21 0)
-			(effects
-				(font
-					(size 1.27 1.27)
-				)
-				(hide yes)
-			)
-		)
-		(pin "1"
-		)
-		(pin "2"
-		)
-		(instances
-			(project "minRead_pcb"
-				(path "/2fbd4c8f-b784-4d80-b374-4947df99a9bf"
-					(reference "R17")
-					(unit 1)
-				)
