File: minRead_pcb.kicad_sch (KiCad schematic)
At the start: 169 parts, among them J1 USB_C_Receptacle, J2 FH34SRJ-24S-0.5SH_50_, J3 FH34SRJ-6S-0.5SH_50_, J4 FH34SRJ-6S-0.5SH_50_, J5 Conn_01x02, J6 PPPC062LJBN-RC, J7 Micro_SD_Card, Q1 FS8205A, Q3 AO3419, Q4 BSS138, Q5 BSS138, Q6 BSS138, Q7 AO3419, Q8 AO3419, SW1 SW_Push, SW10 SW_Push, SW11 SW_Push, SW2 SW_Push, SW3 SW_Push, SW4 SW_Push, SW5 SW_Push, SW6 SW_Push, SW7 SW_Push, SW8 SW_Push, SW9 SW_Push, U1 TPD4E1U06DBVR, U10 TPS923610DRLR, U11 TP4056-42-ESOP8, U12 74LVC1G04, U13 DS3231MZ, U2 TPS2116DRL, U3 AP2112K-3.3, U4 ESP32-S3-WROOM-1, U5 DW01A, U6 TPD4E1U06DBVR, U7 TPD4E1U06DBVR, U8 TPD4E1U06DBVR, U9 TPD4E1U06DBVR

Commit message: Power-path, LED driver and microSD gating fixes from design review
- R17 100k -> 150k: fixes USB_STAT 'on battery' state falling outside its own ADC window
- R38 310k -> 240k: mux switchover was set above the voltage USB_VBUS actually reaches under load (chatter); also makes the ambiguous ST+CHRG state unreachable
- R57/R56 100k/1k -> 1M/10k: cuts unprotected cell drain 41uA -> 4uA
- R75 100k pull-down on COLOR_SEL: 74LVC1G04 input was floating at boot (shoot-through)
- R76 100k pull-down on PWR_BUTTON: internal pull-down is 45k typ with no min/max
- D3 SMAJ30A -> SMAJ26A: 30V part breaks down at 33.3V, above U10's 32V abs max
- R47/R48 4.7k -> 2.2k I2C pull-ups for rise time with the touch FFC attached
- C9 -> 4.7uF, C31 -> 100nF (LED_MONIT settling)
- LED boost moved off the 3V3 rail: U10.VIN -> LDO_IN, Q7 deleted from that role
  (TPS923610 I_SD is 130nA, so the load switch bought nothing)
- microSD power gating: Q7 reused as high-side switch on SD_VDD, all five pull-ups
  and both decaps moved to the switched rail to prevent phantom-powering the card,
  R77 100k bleed, R78 1k gate series, C37 4.7uF -> 1uF (3V3 dip 375mV -> 136mV)
- L1 NR3015T220MNGH is obsolete -> VLS3012HBX-220M annotated
- 50V annotations on the e-paper HV caps
- DESIGN_REVIEW.md: full schematic review with status tracking
Parts:
- added R75, R76, R77: 100k, Resistor_SMD:R_0805_2012Metric_Pad1.20x1.40mm_HandSolder, symbol Device:R
- added R78: 1k, Resistor_SMD:R_0805_2012Metric_Pad1.20x1.40mm_HandSolder, symbol Device:R
- C31: value 10n -> 100n
- C37: value 4.7u -> 1u
- C9: value 1u -> 4.7u
- D3: value SMAJ30A -> SMAJ26A
- R17: value 100k -> 150k
- R38: value 310k -> 240k
- R47, R48: value 4.7k -> 2.2k
- R56: value 1k -> 10k
- R57: value 100k -> 1M
Connections:
- net 3V3: no longer C36.2, C37.2, J7.4 (VDD), R53.2, R54.2, R55.2, R8.2, R9.2
- net COLOR_SEL: now also R75.1
- net GND: now also J6.4, R75.2, R76.2, R77.2; no longer J6.12
- net I2C_SDA: now also J6.8; no longer J6.4
- net LDO_IN: now also C12.2, L2.1, U10.1 (VIN)
- net P+: now also J6.12; no longer J6.8
- net PWR_BUTTON: now also R76.1
- net LED_ACTIVATE: no longer names the net of Q7.1 (G), R40.1
- net LED_ACTIVATE: now also R78.2; no longer U4.34 (IO41)
- new net SD_ACTIVATE: R78.1, U4.34 (IO41)
- new net SD_VDD: C36.2, C37.2, J7.4 (VDD), Q7.3 (D), R53.2, R54.2, R55.2, R77.1, R8.2, R9.2
Other:
- note added: "POWER GATE: SD_ACTIVATE gates VDD to the SD card SD_ACTIVATE HIGH (default) = OFF SD_ACTIVATE LOW = ON All data signals pulled up to SD_VDD All data signals should be asserted low before shutting down"
- note added: "Powered via LDO_IN source instead of 3V3 to reduce stress on LDO output power"
- note added: "Switchover at ~3.4V"
- note added: "VLS3012HBX-220M"
- note removed: "NR3015T220MNGH"
- note removed: "Switchover at ~4.1V"
- moved on the sheet: C36, C37, CR2, CR3, D3, D8, J2, J6, J7, Q7, R40, R53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
