File: minRead_pcb.kicad_sch (KiCad schematic)
At the start: 173 parts, among them J1 USB_C_Receptacle, J2 FH34SRJ-24S-0.5SH_50_, J3 FH34SRJ-6S-0.5SH_50_, J4 FH34SRJ-6S-0.5SH_50_, J5 Conn_01x02, J6 PPPC062LJBN-RC, J7 Micro_SD_Card, Q1 FS8205A, Q3 AO3419, Q4 BSS138, Q5 BSS138, Q6 BSS138, Q7 AO3419, Q8 AO3419, SW1 SW_Push, SW10 SW_Push, SW11 SW_Push, SW2 SW_Push, SW3 SW_Push, SW4 SW_Push, SW5 SW_Push, SW6 SW_Push, SW7 SW_Push, SW8 SW_Push, SW9 SW_Push, U1 TPD4E1U06DBVR, U10 TPS923610DRLR, U11 TP4056-42-ESOP8, U12 74LVC1G04, U13 DS3231MZ, U2 TPS2116DRL, U3 AP2112K-3.3, U4 ESP32-S3-WROOM-1, U5 DW01A, U6 TPD4E1U06DBVR, U7 TPD4E1U06DBVR, U8 TPD4E1U06DBVR, U9 TPD4E1U06DBVR

Commit message: Add Silkscreen hardware documentation; ERC clean, J6 re-ordered
docs/HARDWARE.md: full block-by-block explanation of the board with
annotated schematic screenshots (23 images cropped from the plotted PDF).
Covers the power chain, MCU, SDMMC, e-paper interface and charge pump,
frontlight driver, touch, button ladders, RTC and expansion header,
plus a complete GPIO map and the four 'agnostic' design goals.

Explicitly framed as post-hoc documentation for review/tweaking - it was
not used to design the board.

Schematic changes in this commit:
- ERC now reports 0 errors (was 4): TPS923610 GND pin retyped to
  power_input, #FLG05 removed from LDO_IN, PWR_FLAG added to SD_VDD
- J6 re-ordered so LED_SW is bounded only by GND/W-/C- and P+ sits in
  the corner next to the LED returns; SDA moved to pin 8, GND to pin 4
- J2 symbol pin names corrected (pin 4 is NC; VGH/VGL/VSH/VSL now read
  correctly against the panel datasheet)
- 50V ratings appended to the e-paper HV capacitor values
- L1 replacement annotated (NR3015T220MNGH is obsolete -> VLS3012HBX-220M)
- stale 'Switchover at ~4.1V' note corrected to ~3.4V

DESIGN_REVIEW.md: status updated for the above; new section 6.16 records
that LED_MONIT reads ~0.25-0.46 V rather than 0 V when the frontlight is
disabled, because the boost body-diode path holds LED_SW near LDO_IN.
Parts:
- C13, C14, C15, C16, C9: value 4.7u -> 4.7u/50V
- C20: value 1u -> 1u/50V
Other:
- moved on the sheet: C36, C37

Commit message: Downsize passives to 0603, document D1 redundancy and layout guidance
Schematic:
- Swap 78 resistors and 22 capacitors from 0805 to 0603 hand-solder
  footprints, recovering ~228 mm^2 of courtyard. F1 (fuse) and D2 (LED)
  untouched. 13 capacitors deliberately kept at 0805.
- C11 and C17 annotated /50V, closing the HV cap rating gap.

DESIGN_REVIEW.md:
- 6.19: 0805->0603 migration audit. Corrected an earlier power analysis
  that wrongly assumed full rail voltage across every resistor; real
  worst case is R14 at 28 mW (28% of an 0603). Verified 0603 MLCC
  ceilings against manufacturer catalogs and LCSC stock: 4.7uF/50V does
  not exist in 0603, and 22uF/6.3V delivers only 6.7uF at 3.3V bias.
- 6.20: D1 (series Schottky on VBUS) is redundant. TPS2116 specifies
  1 nA reverse leakage out of an unselected input; the TP4056 datasheet
  states outright that no blocking diode is required. D1 costs 0.3-0.6 V
  of headroom, exceeds its SOD-123 500 mW rating at the current F1 will
  pass, and blocks raising R38 to close the LDO brown-out window.
- 3.3: withdrew the earlier "raise C9 to 4.7uF" recommendation. Ripple
  at 1.1 MHz is optically invisible and R37 dominates the loop, while
  larger C9 slows CCT blending worst at low brightness. 1 uF is correct.
- 8: new placement and layout guidance for the 2-layer stackup, covering
  the two switching loops, thermal separation of U3/U11, analog routing,
  and the antenna keepout.

docs/HARDWARE.md:
- Note D1 under review; document the 0603/0805 split and its rationale.

Add .gitignore rules for KiCad autosave, lock and backup files.

ERC: 0 errors, 40 cosmetic warnings. Netlist verified at 170 components
and 127 nets after the footprint swap.
Parts:
- removed TP3, TP4, TP5: TestPoint, Connector_PinHeader_2.54mm:PinHeader_1x01_P2.54mm_Vertical, symbol Connector:TestPoint
- C1, C10, C12, C2, C21, C22, C23, C24, C25, C26, C27, C28, C29, C3, C30, C31, C33, C36, C37, C5, C7, C8: footprint Capacitor_SMD:C_0805_2012Metric_Pad1.18x1.45mm_HandSolder -> Capacitor_SMD:C_0603_1608Metric_Pad1.08x0.95mm_HandSolder
- C11, C17: value 4.7u -> 4.7u/50V
- C9: value 4.7u/50V -> 1u/50V
- R1, R10, R11, R12, R13, R14, R15, R16, R17, R18, R19, R2, R20, R21, R22, R23, R24, R25, R26, R27, R28, R29, R3, R30, R31, R32, R33, R34, R35, R36, R37, R38, R39, R4, R40, R41, R42, R43, R44, R45, R46, R47, R48, R49, R5, R50, R51, R52, R53, R54, R55, R56, R57, R58, R59, R6, R60, R61, R62, R63, R64, R65, R66, R67, R68, R69, R7, R70, R71, R72, R73, R74, R75, R76, R77, R78, R8, R9: footprint Resistor_SMD:R_0805_2012Metric_Pad1.20x1.40mm_HandSolder -> Resistor_SMD:R_0603_1608Metric_Pad0.98x0.95mm_HandSolder
Connections:
- net IO35_PSRAM: no longer names the net of U4.28 (IO35)
- net IO36_PSRAM: no longer names the net of U4.29 (IO36)
- net IO37_PSRAM: no longer names the net of U4.30 (IO37)
- no-connect marks 12 -> 15
Other:
- note removed: "ESP32-S31-WROOM-1 does not reserve GPIO for PSRAM Future proofing :)"

Commit message: Remove D1, raise charge current, reassign 6 GPIOs, begin layout
Schematic:
- Remove D1 (series Schottky on VBUS) and raise R38 to 300k. F1 now
  feeds USB_VBUS directly. Switchover threshold becomes 3.68/4.00/4.32 V,
  clearing the AP2112K's 3.72 V requirement while holding +0.22 V margin
  at 1 A. Recovers 0.3-0.6 V of rail headroom and removes 200-600 mW of
  dissipation from a part rated 500 mW.
- R6 12k -> 4.7k, raising TP4056 charge current from ~100 mA to ~255 mA.
  Worst-case charger dissipation ~500 mW at a depleted cell, about +20 C
  on the ESOP-8 thermal pad. Well inside the 125 C regulation point.
- Reassign 6 ESP32 pins to shorten routes: IO9 LED_MONIT->USB_STAT,
  IO10 TP_INT->SD_ACTIVATE, IO40 PWM_LED->COLOR_SEL, IO41
  SD_ACTIVATE->TP_INT, IO42 COLOR_SEL->PWM_LED, IO2 USB_STAT->LED_MONIT.
  All five analog nets remain on ADC1, no strapping pins disturbed, and
  moving PWM_LED onto IO42 is safer than COLOR_SEL was since the ~60 us
  power-up glitch now means "LED off" rather than an unintended CCT state.

Layout:
- Placement pass: 124 of 170 footprints repositioned.
- Routing begun: 328 track segments and 18 vias.

Docs:
- DESIGN_REVIEW 6.20.7 marked implemented; new 6.21 (charge current) and
  6.22 (GPIO reassignment, with the ADC1 and strapping-pin verification).
- HARDWARE.md GPIO map and all inline pin references updated to match;
  every row cross-checked against the regenerated netlist.
- Flag one regression: C11 lost its /50V annotation while C13-C17 and
  C20 kept theirs. C11 is the charge-pump flying capacitor and swings
  the full 0-23 V every cycle, so it is the one that least deserves to
  lose its rating.

ERC: 0 errors, 40 cosmetic warnings. 169 components, 126 nets.
Parts:
- removed D1: B5819W, Diode_SMD:D_SOD-123, symbol Diode:MBR0530
- C11: value 4.7u/50V -> 4.7u
- R38: value 240k -> 300k
- R6: value 12k -> 4.7k
Connections:
- net COLOR_SEL: now also U4.33 (IO40); no longer U4.35 (IO42)
- net LED_MONIT: now also U4.38 (IO2); no longer U4.17 (IO9)
- net PIN_5: now also R45.2; no longer R58.2
- net PIN_6: now also R58.2; no longer R45.2
- net PWM_LED: now also U4.35 (IO42); no longer U4.33 (IO40)
- net SD_ACTIVATE: now also U4.18 (IO10); no longer U4.34 (IO41)
- net TP_INT: now also U4.34 (IO41); no longer U4.18 (IO10)
- net USB_STAT: now also U4.17 (IO9); no longer U4.38 (IO2)
- net USB_VBUS: now also F1.2
Other:
- note added: "R6 4.7kohm -> 255mA charge rate"
- note added: "used to be a schottky diode on VBUS but removed due to tp4056 blocking reverse current"
- note removed: "R6 12kohm -> 100mA charge rate"
Changed lines of the file:
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@@
 		)
 	)
-	(text "R6 12kohm -> 100mA charge rate"
+	(text "R6 4.7kohm -> 255mA charge rate"
 		(exclude_from_sim no)
 		(at 149.098 123.952 0)
@@
 		)
 	)
+	(text "used to be a schottky diode on VBUS \nbut removed due to tp4056 blocking reverse \ncurrent"
+		(exclude_from_sim no)
+		(at 63.754 68.834 0)
+		(effects
+			(font
+				(size 1.27 1.27)
+			)
+		)
+	)
 	(text_box "TPS923 chip is a series LED boost converter. \nRecommended to run between 10kHz-25kHz via PWM_LED for brightness control.\nReturn path for LEDs is toggled via COLOR_SEL for warm/cool selection.\nFeedback current is 15mA tuned via R37. Reference datasheet to change as needed.\nLED_MONIT is analog signal that references 0-24.5V output on LED voltage. (ADC range from 0 to ~30V)\nInternal OVP should cut out at ~24V, but software protection should kick in and disable LED_ACTIVATE at safe voltage above known forward voltage (15V)"
 		(exclude_from_sim no)
@@
 	(wire
 		(pts
-			(xy 57.15 30.48) (xy 58.42 30.48)
+			(xy 57.15 30.48) (xy 67.31 30.48)
 		)
 		(stroke
@@
 	(wire
 		(pts
-			(xy 66.04 30.48) (xy 67.31 30.48)
-		)
-		(stroke
-			(width 0)
-			(type default)
-		)
-	)
-	(wire
-		(pts
 			(xy 247.65 102.87) (xy 247.65 110.49)
 		)
@@
 		)
 	)
-	(label "PIN_5"
+	(label "PIN_6"
 		(at 355.6 393.7 0)
 		(effects
@@
 		)
 	)
-	(label "PIN_6"
+	(label "PIN_5"
 		(at 355.6 387.35 0)
 		(effects
@@
 	(global_label "SD_ACTIVATE"
 		(shape input)
-		(at 514.35 217.17 0)
+		(at 483.87 214.63 180)
 		(fields_autoplaced yes)
 		(effects
@@
 				(size 1.27 1.27)
 			)
-			(justify left)
+			(justify right)
 		)
 		(property "Intersheetrefs" "${INTERSHEET_REFS}"
-			(at 529.0071 217.17 0)
+			(at 469.2129 214.63 0)
 			(effects
 				(font
 					(size 1.27 1.27)
 				)
-				(justify left)
+				(justify right)
 				(hide yes)
 			)
@@
 	(global_label "LED_MONIT"
 		(shape input)
-		(at 483.87 212.09 180)
+		(at 483.87 194.31 180)
 		(fields_autoplaced yes)
 		(effects
@@
 		)
 		(property "Intersheetrefs" "${INTERSHEET_REFS}"
-			(at 470.7853 212.09 0)
+			(at 470.7853 194.31 0)
 			(effects
 				(font
@@
 	(global_label "TP_INT"
 		(shape input)
-		(at 483.87 214.63 180)
+		(at 514.35 217.17 0)
 		(fields_autoplaced yes)
 		(effects
@@
 				(size 1.27 1.27)
 			)
-			(justify right)
+			(justify left)
 		)
 		(property "Intersheetrefs" "${INTERSHEET_REFS}"
-			(at 474.7767 214.63 0)
+			(at 523.4433 217.17 0)
 			(effects
 				(font
 					(size 1.27 1.27)
 				)
-				(justify right)
+				(justify left)
 				(hide yes)
 			)
@@
 	(global_label "PWM_LED"
 		(shape input)
-		(at 514.35 214.63 0)
+		(at 514.35 219.71 0)
 		(fields_autoplaced yes)
 		(effects
@@
 		)
 		(property "Intersheetrefs" "${INTERSHEET_REFS}"
-			(at 525.9227 214.63 0)
+			(at 525.9227 219.71 0)
 			(effects
 				(font
@@
 	(global_label "COLOR_SEL"
 		(shape input)
-		(at 514.35 219.71 0)
+		(at 514.35 214.63 0)
 		(fields_autoplaced yes)
 		(effects
@@
 		)
 		(property "Intersheetrefs" "${INTERSHEET_REFS}"
-			(at 527.9185 219.71 0)
+			(at 527.9185 214.63 0)
 			(effects
 				(font
@@
 	(global_label "USB_STAT"
 		(shape input)
-		(at 483.87 194.31 180)
+		(at 483.87 212.09 180)
 		(fields_autoplaced yes)
 		(effects
@@
 		)
 		(property "Intersheetrefs" "${INTERSHEET_REFS}"
-			(at 471.8739 194.31 0)
+			(at 471.8739 212.09 0)
 			(effects
 				(font
@@
 			)
 		)
-		(property "Value" "240k"
+		(property "Value" "300k"
 			(at 163.83 52.0699 0)
 			(effects
@@
 	)
 	(symbol
-		(lib_id "Diode:MBR0530")
-		(at 62.23 30.48 180)
-		(unit 1)
-		(exclude_from_sim no)
-		(in_bom yes)
-		(on_board yes)
-		(dnp no)
-		(property "Reference" "D1"
-			(at 62.738 24.892 0)
-			(effects
-				(font
-					(size 1.27 1.27)
-				)
-			)
-		)
-		(property "Value" "B5819W"
-			(at 63.246 27.178 0)
-			(effects
-				(font
-					(size 1.27 1.27)
-				)
-			)
-		)
-		(property "Footprint" "Diode_SMD:D_SOD-123"
-			(at 62.23 26.035 0)
-			(effects
-				(font
-					(size 1.27 1.27)
-				)
-				(hide yes)
-			)
-		)
-		(property "Datasheet" "http://www.mccsemi.com/up_pdf/MBR0520~MBR0580(SOD123).pdf"
-			(at 62.23 30.48 0)
-			(effects
-				(font
-					(size 1.27 1.27)
-				)
-				(hide yes)
-			)
-		)
-		(property "Description" "30V 0.5A Schottky Power Rectifier Diode, SOD-123"
-			(at 62.23 30.48 0)
-			(effects
-				(font
-					(size 1.27 1.27)
-				)
-				(hide yes)
-			)
-		)
-		(pin "2"
-		)
-		(pin "1"
-		)
-		(instances
-			(project "minRead_pcb"
-				(path "/2fbd4c8f-b784-4d80-b374-4947df99a9bf"
-					(reference "D1")
-					(unit 1)
-				)
-			)
-		)
-	)
-	(symbol
 		(lib_id "Device:R")
 		(at 532.13 113.03 180)
@@
 			)
 		)
-		(property "Value" "12k"
+		(property "Value" "4.7k"
 			(at 142.24 110.4899 0)
 			(effects
@@
 			)
 		)
-		(property "Value" "4.7u/50V"
+		(property "Value" "4.7u"
 			(at 55.88 292.1 90)
 			(effects

Commit message: Layout pass + full documentation sync
Layout (minRead_pcb.kicad_pcb / .kicad_sch / .kicad_pro):
- 2-layer layout completed and routed (0 unconnected); DRC clean apart
  from cosmetic silkscreen, benign starved-GND thermals, and the J1
  connector clearance (5 V pads vs the 0.20 mm Power class)
- silkscreen cleanup and reference-designator sizing normalised
- both switching nodes tightened: LED boost hot loop (U10.VOUT->C9->GND)
  with C9 on-side and on-top; e-ink EINK_SW collapsed from a plane to a
  compact node
- added frontlight test points TP3-TP5 (LED_SW / C- / W-) and a 5th
  mounting hole; board now 173 components / 126 nets

Docs (DESIGN_REVIEW.md, docs/HARDWARE.md) synced to as-built:
- LDO swapped AP2112K-3.3 -> TLV75533P (25 uA Iq); §3.2/§6.20/§6.23
  re-evaluated with the lower-dropout part in place
- D1 removed, R38 = 300 k (switchover 3.68/4.00/4.32 V); R6 = 4.7 k
  (~255 mA charge); C11 restored to 4.7u/50V; J2 pin 5 = VSH2
- USB_STAT re-done from scratch: ST reports mux source (not USB
  presence), ST+CHRG is a decodable/benign weak-source diagnostic, plus
  firmware decode windows; documented why it can't be designed out at
  300 k (V_REF spread > LDO/charger guard band)
- test-point, mounting-hole and component/net counts updated (173/126);
  §8 marked layout-done with a coordinate-level spot-review summary
Parts:
- removed U3: AP2112K-3.3, Package_TO_SOT_SMD:SOT-23-5_HandSoldering, symbol Regulator_Linear:AP2112K-3.3
- added H5: MountingHole_Pad, MountingHole:MountingHole_2.2mm_M2_DIN965_Pad_TopBottom, symbol Mechanical:MountingHole_Pad
- added TP3, TP4, TP5: TestPoint, Connector_PinHeader_2.54mm:PinHeader_1x01_P2.54mm_Vertical, symbol Connector:TestPoint
- added U14: TLV75533PDBV, Package_TO_SOT_SMD:SOT-23-5_HandSoldering, symbol Regulator_Linear:TLV75533PDBV
- C11: value 4.7u -> 4.7u/50V
- renumbered R25 to R24, R24 to R25
Connections:
- net 3V3: now also U14.5 (OUT)
- net C-: now also TP4.1
- net GND: now also H5.1, U14.2 (GND)
- net LDO_IN: now also U14.1 (IN), U14.3 (EN)
- net LED_SW: now also TP3.1
- net SD_CLK: now also U1.4; no longer U9.1
- net SD_CMD: now also U1.6; no longer U9.3
- net SD_DAT0: now also U9.3; no longer U1.6
- net SD_DAT1: now also U9.1; no longer U1.4
- net W-: now also TP5.1
- net VBUS_PRE renamed VBUS_PRE_FUSE
