File: silkscreen_pcb.kicad_pcb (KiCad board)
At the start: 2 copper layers, 60 x 111.3 mm, 176 parts, among them J1 USB_C_Receptacle, J2 FH34SRJ-24S-0.5SH_50_, J3 FH34SRJ-6S-0.5SH_50_, J4 FH34SRJ-6S-0.5SH_50_, J5 Conn_01x02, J6 PPPC062LJBN-RC, J7 Micro_SD_Card, Q1 FS8205A, Q3 AO3419, Q4 BSS138, Q5 BSS138, Q6 BSS138, Q7 AO3419, Q8 AO3419, SW1 SW_Push, SW10 SW_Push, SW11 SW_Push, SW2 SW_Push, SW3 SW_Push, SW4 SW_Push, SW5 SW_Push, SW6 SW_Push, SW7 SW_Push, SW8 SW_Push, SW9 SW_Push, U1 TPD4E1U06DBVR, U10 TPS923610DRLR, U11 TP4056-42-ESOP8, U12 74LVC1G04, U13 DS3231MZ, U14 TLV75533PDBV, U2 TPS2116DRL, U4 ESP32-S3-WROOM-1, U5 DW01A, U6 TPD4E1U06DBVR, U7 TPD4E1U06DBVR, U8 TPD4E1U06DBVR, U9 TPD4E1U06DBVR

Commit message: Rename project to silkscreen_pcb; add README, CERN-OHL-S license, fab/BOM
- rename minRead_pcb.{kicad_pro,kicad_sch,kicad_pcb} -> silkscreen_pcb.*
  and update all internal project-name references + doc references
- add top-level README.md (board overview, fab/assembly how-to, license)
- add LICENSE: CERN Open Hardware Licence v2 - Strongly Reciprocal
  (CERN-OHL-S-2.0), full verbatim text
- fabrication/: full BOM (BOM.md/BOM.csv) with manufacturers, MPNs,
  DigiKey/LCSC links, LCSC-cheaper alternates and per-part pricing +
  a complete-build cost section; JLC-format BOM/CPL; generic centroid;
  and a per-house how-to (README.md)
- gitignore generated gerbers/drill and the gerber zip (regenerate via
  kicad-cli; BOM + assembly data + how-to remain tracked)

Note: the LDO is U3 (TLV75533P), consistent with the docs.
Parts:
- renumbered U14 to U3

Commit message: Remove unused/redundant third-party libraries; title-block + silkscreen edits
- delete unused vendored library folders: BQ24074RGTR, TPD4E004DRYR,
  TPD6E004RSER, sfv24r (unused SnapEDA parts); PPTC042/052/062LFBN
  (unused Sullins header libs); USB4085_GF_A (J1 uses the KiCad-standard
  USB-C footprint)
- delete redundant Battery_Management (byte-identical to KiCad's stock
  library; DW01A/TP4056 resolve to the standard lib)
- prune sym-lib-table (13->8) and fp-lib-table (13->8) to the used
  vendored libraries only; all remaining URIs verified
- title-block and silkscreen edits
Parts:
- added G***: LOGO, LOGO, F.Cu at (51.4, 136.1)
- moved G*** 3.42 mm to (82.2, 136.1)
- moved G*** 3.42 mm to (92.2, 136.1)
- moved G*** 3.42 mm to (72.2, 136.1)
Routing:
- net C-: vias 5 -> 4
Other:
- board text added: "made with love by Ian C supported by several, including:"
- board text removed: "cat by @tomisit0"
- board text removed: "made with love by Ian C supported by many, including:"
