File: silkscreen_pcb.kicad_pcb (KiCad board)
At the start: 2 copper layers, 60 x 111.3 mm, 177 parts, among them J1 USB_C_Receptacle, J2 FH34SRJ-24S-0.5SH_50_, J3 FH34SRJ-6S-0.5SH_50_, J4 FH34SRJ-6S-0.5SH_50_, J5 Conn_01x02, J6 PPPC062LJBN-RC, J7 Micro_SD_Card, Q1 FS8205A, Q3 AO3419, Q4 BSS138, Q5 BSS138, Q6 BSS138, Q7 AO3419, Q8 AO3419, SW1 SW_Push, SW10 SW_Push, SW11 SW_Push, SW2 SW_Push, SW3 SW_Push, SW4 SW_Push, SW5 SW_Push, SW6 SW_Push, SW7 SW_Push, SW8 SW_Push, SW9 SW_Push, U1 TPD4E1U06DBVR, U10 TPS923610DRLR, U11 TP4056-42-ESOP8, U12 74LVC1G04, U13 DS3231MZ, U2 TPS2116DRL, U3 TLV75533PDBV, U4 ESP32-S3-WROOM-1, U5 DW01A, U6 TPD4E1U06DBVR, U7 TPD4E1U06DBVR, U8 TPD4E1U06DBVR, U9 TPD4E1U06DBVR

Commit message: Docs pass: current plots + board render; confirm L2 MPN
- add current full plots to docs/ (silkscreen_pcb_schematic.pdf,
  silkscreen_pcb.pdf) and link them from README and HARDWARE.md as the
  authoritative up-to-date views
- add a 3D board render (docs/images/board-3d-top.png) to the README
- note in HARDWARE.md that the per-block screenshots may lag the latest
  revision (the PDFs are authoritative)
- BOM: L2 = Würth 74479325207247 (confirmed); drop the resolved
  "verify L2 MPN" caveat; DESIGN_REVIEW §3.5 updated to match
- includes title-block / silkscreen edits in the .kicad files

Verified against the live netlist: GPIO map, counts (173/126) and refs
(LDO = U3/TLV75533P) are all current.
Routing:
- net W-: track 189.8 -> 191.9 mm
- net C-: track 217.3 -> 219.3 mm
- net UNUSED_GPIO_3: track 67.7 -> 69.5 mm
- net I2C_SDA: track 184.3 -> 183.1 mm
- net LED_SW: track 197.8 -> 198.3 mm
- net GND: vias 45 -> 46
Other:
- outline, holes or cut-outs redrawn
